File: NFCPower10.kicad_pcb (KiCad board)
At the start: 2 copper layers, 270 x 125 mm, 601 parts, among them J1 PJ-002AH, J10 SSW-102-01-T-S, J11 SSW-102-01-T-S, J12 Conn_02x03_Odd_Even, J13 SSW-102-01-T-S, J14 SSW-102-01-T-S, J15 Conn_02x03_Odd_Even, J16 SSW-102-01-T-S, J17 SSW-102-01-T-S, J18 Conn_02x03_Odd_Even, J19 SSW-102-01-T-S, J2 475890001, J20 SSW-102-01-T-S, J21 Conn_02x03_Odd_Even, J22 SSW-102-01-T-S, J23 SSW-102-01-T-S, J24 Conn_02x03_Odd_Even, J25 SSW-102-01-T-S, J26 SSW-102-01-T-S, J27 Conn_02x03_Odd_Even, J28 SSW-102-01-T-S, J29 SSW-102-01-T-S, J3 Conn_02x03_Odd_Even, J30 Conn_02x03_Odd_Even, J31 SSW-102-01-T-S, J32 SSW-102-01-T-S, J33 Conn_02x03_Odd_Even, J34 SSW-102-01-T-S, J35 SSW-102-01-T-S, J4 SSW-104-01-T-S, J5 SSW-106-02-T-S, J6 Conn_02x03_Odd_Even, J7 SSW-102-01-T-S, J8 SSW-102-01-T-S, J9 Conn_02x03_Odd_Even, Q1 BSS138, Q2 BSS138, Q3 BSS138, Q4 BSS138, Q5 BSS138, SW1 FSM2JSMAA, SW2 FSM2JSMAA, U1 ATMEGA328P-MU, U10 ATMEGA328P-MU, U11 ST25R3916-AQWT, U12 ATMEGA328P-MU, U13 ST25R3916-AQWT, U14 ATMEGA328P-MU, U15 ST25R3916-AQWT, U16 ATMEGA328P-MU, U17 ST25R3916-AQWT, U18 ATMEGA328P-MU, U19 ST25R3916-AQWT, U2 FT231XQ-R, U20 ATMEGA328P-MU, U21 ST25R3916-AQWT, U22 ATMEGA328P-MU, U23 ST25R3916-AQWT, U3 Si5351A-B-GM, U4 ATMEGA328P-MU, U5 ST25R3916-AQWT, U6 ATMEGA328P-MU, U7 ST25R3916-AQWT, U8 ATMEGA328P-MU, U9 ST25R3916-AQWT, Y1 TSX-3225_16.0000MF09Z-AC3, Y10 Coil_49_18_6T_2Layer, Y11 Field_Sensor_54_22, Y12 TSX-3225_16.0000MF09Z-AC3, Y13 Coil_49_18_6T_2Layer, Y14 Field_Sensor_54_22, Y15 TSX-3225_16.0000MF09Z-AC3, Y16 Coil_49_18_6T_2Layer, Y17 Field_Sensor_54_22, Y18 TSX-3225_16.0000MF09Z-AC3, Y19 Coil_49_18_6T_2Layer, Y2 ABM8G-25.000MHz-B4Y-T, Y20 Field_Sensor_54_22, Y21 TSX-3225_16.0000MF09Z-AC3, Y22 Coil_49_18_6T_2Layer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

Commit message: initial placement
Parts:
- added REF**: MountingHole_3.2mm_M3, Mounting_Holes:MountingHole_3.2mm_M3, F.Cu at (343.5, 200.0)
- added REF**: MountingHole_3.2mm_M3, Mounting_Holes:MountingHole_3.2mm_M3, F.Cu at (343.5, 85.0)
- added REF**: MountingHole_3.2mm_M3, Mounting_Holes:MountingHole_3.2mm_M3, F.Cu at (83.5, 85.0)
- added REF**: MountingHole_3.2mm_M3, Mounting_Holes:MountingHole_3.2mm_M3, F.Cu at (83.5, 200.0)
- Y11, Y14, Y17, Y20, Y23, Y26, Y29, Y32, Y5, Y8: moved to B.Cu
- moved C286 418.4 mm to (90.9, 141.0), turned to 180 degrees
- moved C280 407.8 mm to (93.0, 160.0), turned to 180 degrees
- moved C271 403.5 mm to (104.5, 144.5)
- moved C274 402.9 mm to (101.5, 144.5), turned to 180 degrees
- moved J6 402.8 mm to (333.5, 172.4)
- moved C273 402.2 mm to (104.5, 142.5)
- moved C287 401.6 mm to (108.5, 138.5)
- moved C276 399.7 mm to (101.5, 142.5), turned to 180 degrees
- moved C282 398.9 mm to (93.0, 154.0)
- moved C270 394.9 mm to (108.5, 145.5)
- moved D63 394.7 mm to (93.0, 145.5)
- moved C277 394.6 mm to (108.5, 147.5)
- moved U22 394.2 mm to (101.0, 164.5)
- moved C285 394.1 mm to (97.5, 156.0)
- moved C266 393.0 mm to (104.5, 156.0)
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Connections:
- C120 pad 1: /TX4/RF1 -> /TX4/RF2
- C121 pad 2: /TX4/RF2 -> /TX4/RF1
- C122 pad 1: /TX4/RF1 -> /TX4/RF2
- C148 pad 1: /TX5/RF1 -> /TX5/RF2
- C149 pad 2: /TX5/RF2 -> /TX5/RF1
- C150 pad 1: /TX5/RF1 -> /TX5/RF2
- C176 pad 1: /TX6/RF1 -> /TX6/RF2
- C177 pad 2: /TX6/RF2 -> /TX6/RF1
- C178 pad 1: /TX6/RF1 -> /TX6/RF2
- C204 pad 1: /TX7/RF1 -> /TX7/RF2
- C205 pad 2: /TX7/RF2 -> /TX7/RF1
- C206 pad 1: /TX7/RF1 -> /TX7/RF2
- C232 pad 1: /TX8/RF1 -> /TX8/RF2
- C233 pad 2: /TX8/RF2 -> /TX8/RF1
- C234 pad 1: /TX8/RF1 -> /TX8/RF2
- C260 pad 1: /TX9/RF1 -> /TX9/RF2
- C261 pad 2: /TX9/RF2 -> /TX9/RF1
- C262 pad 1: /TX9/RF1 -> /TX9/RF2
- C288 pad 1: /TX10/RF1 -> /TX10/RF2
- C289 pad 2: /TX10/RF2 -> /TX10/RF1
- C290 pad 1: /TX10/RF1 -> /TX10/RF2
- C36 pad 1: /TX1/RF1 -> /TX1/RF2
- C37 pad 2: /TX1/RF2 -> /TX1/RF1
- C38 pad 1: /TX1/RF1 -> /TX1/RF2
- C64 pad 1: /TX2/RF1 -> /TX2/RF2
- C65 pad 2: /TX2/RF2 -> /TX2/RF1
- C66 pad 1: /TX2/RF1 -> /TX2/RF2
- C92 pad 1: /TX3/RF1 -> /TX3/RF2
- C93 pad 2: /TX3/RF2 -> /TX3/RF1
- C94 pad 1: /TX3/RF1 -> /TX3/RF2
- L1 pad 1: /TX1/RFO1 -> /TX1/RFO2
- L1 pad 2: /TX1/RF1 -> /TX1/RF2
- L10 pad 1: /TX5/RFO2 -> /TX5/RFO1
- L10 pad 2: /TX5/RF2 -> /TX5/RF1
- L11 pad 1: /TX6/RFO1 -> /TX6/RFO2
- L11 pad 2: /TX6/RF1 -> /TX6/RF2
- L12 pad 1: /TX6/RFO2 -> /TX6/RFO1
- L12 pad 2: /TX6/RF2 -> /TX6/RF1
- L13 pad 1: /TX7/RFO1 -> /TX7/RFO2
- L13 pad 2: /TX7/RF1 -> /TX7/RF2
- L14 pad 1: /TX7/RFO2 -> /TX7/RFO1
- L14 pad 2: /TX7/RF2 -> /TX7/RF1
- L15 pad 1: /TX8/RFO1 -> /TX8/RFO2
- L15 pad 2: /TX8/RF1 -> /TX8/RF2
- L16 pad 1: /TX8/RFO2 -> /TX8/RFO1
- L16 pad 2: /TX8/RF2 -> /TX8/RF1
- L17 pad 1: /TX9/RFO1 -> /TX9/RFO2
- L17 pad 2: /TX9/RF1 -> /TX9/RF2
- L18 pad 1: /TX9/RFO2 -> /TX9/RFO1
- L18 pad 2: /TX9/RF2 -> /TX9/RF1
- L19 pad 1: /TX10/RFO1 -> /TX10/RFO2
- L19 pad 2: /TX10/RF1 -> /TX10/RF2
- L2 pad 1: /TX1/RFO2 -> /TX1/RFO1
- L2 pad 2: /TX1/RF2 -> /TX1/RF1
- L20 pad 1: /TX10/RFO2 -> /TX10/RFO1
- L20 pad 2: /TX10/RF2 -> /TX10/RF1
- L3 pad 1: /TX2/RFO1 -> /TX2/RFO2
- L3 pad 2: /TX2/RF1 -> /TX2/RF2
- L4 pad 1: /TX2/RFO2 -> /TX2/RFO1
- L4 pad 2: /TX2/RF2 -> /TX2/RF1
- L5 pad 1: /TX3/RFO1 -> /TX3/RFO2
- L5 pad 2: /TX3/RF1 -> /TX3/RF2
- L6 pad 1: /TX3/RFO2 -> /TX3/RFO1
- L6 pad 2: /TX3/RF2 -> /TX3/RF1
- L7 pad 1: /TX4/RFO1 -> /TX4/RFO2
- L7 pad 2: /TX4/RF1 -> /TX4/RF2
- L8 pad 1: /TX4/RFO2 -> /TX4/RFO1
- L8 pad 2: /TX4/RF2 -> /TX4/RF1
- L9 pad 1: /TX5/RFO1 -> /TX5/RFO2
- L9 pad 2: /TX5/RF1 -> /TX5/RF2
- Y10 pad 2: /TX3/RF2 -> /TX3/RF1
- Y13 pad 2: /TX4/RF2 -> /TX4/RF1
- Y16 pad 2: /TX5/RF2 -> /TX5/RF1
- Y19 pad 2: /TX6/RF2 -> /TX6/RF1
- Y22 pad 2: /TX7/RF2 -> /TX7/RF1
- Y25 pad 2: /TX8/RF2 -> /TX8/RF1
- Y28 pad 2: /TX9/RF2 -> /TX9/RF1
- Y31 pad 2: /TX10/RF2 -> /TX10/RF1
- Y4 pad 2: /TX1/RF2 -> /TX1/RF1
- Y7 pad 2: /TX2/RF2 -> /TX2/RF1
Other:
- board text added: "5V/3A"
- board text added: "CS SCK MOSI MISO +5V GND"
- board text added: "GND MOSI +5V"
- board text added: "GOOD"
- board text added: "HSEN1"
- board text added: "HSEN2"
- board text added: "ISP"
- board text added: "Interrupt"
- board text added: "NFCPower10 - YSO"
- board text added: "OLED Display I2C Port"
- board text added: "OPEN"
- board text added: "RED"
- board text added: "RES SCK MISO"
- board text added: "RF ON"
- board text added: "RX"
- board text added: "RXP"
- board text added: "Reset"
- board text added: "SCK"
- board text added: "SD Card SPI Port"
- board text added: "SDA SCL +5V GND"
- board text added: "SHORT"
- board text added: "TX"
- board text added: "TX1"
- board text added: "TX10"
- board text added: "TX2"
- board text added: "TX3"
- board text added: "TX4"
- board text added: "TX5"
- board text added: "TX6"
- board text added: "TX7"
- board text added: "TX8"
- board text added: "TX9"
- board text added: "TXP"

Commit message: initial routing
Routing:
- net GND: track 0.00 -> 1063.3 mm, vias 0 -> 164
- net +5VP: track 0.00 -> 930.4 mm, vias 0 -> 50
- net +5V: track 0.00 -> 278.2 mm, vias 0 -> 10
- net /SDAP: track 0.00 -> 142.7 mm, vias 0 -> 20
- net /SDA: track 0.00 -> 125.3 mm, vias 0 -> 6
- net /SCLP: track 0.00 -> 121.7 mm
- net /SCL: track 0.00 -> 118.3 mm, vias 0 -> 4
- net /TX: track 0.00 -> 97.1 mm, vias 0 -> 6
- net /OEB: track 0.00 -> 96.0 mm, vias 0 -> 4
- net /IRQ: track 0.00 -> 92.5 mm, vias 0 -> 4
- net /SSEN: track 0.00 -> 91.7 mm, vias 0 -> 4
- net /RES: track 0.00 -> 69.7 mm, vias 0 -> 1
- net /TX3/RES: track 0.00 -> 46.3 mm, vias 0 -> 2
- net /TX2/RES: track 0.00 -> 46.3 mm, vias 0 -> 2
- net /TX1/RES: track 0.00 -> 46.3 mm, vias 0 -> 2
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- added copper zone on B.Cu, net GND
Other:
- net class Default: clearance 0.2 -> 0.1524
- rule trace_clearance: 0.2 -> 0.1524

Commit message: continue routing. add INA219 to monitor +5VP rail.
Parts:
- added R16: RL2512FK-070R1L, project:YAGEO-RL2512-02_2018-10-MFG, F.Cu at (213.5, 187.2)
- added REF**: Fiducial_1mm_Dia_2.54mm_Outer_CopperTop, Fiducials:Fiducial_1mm_Dia_2.54mm_Outer_CopperTop, F.Cu at (83.5, 91.0)
- added REF**: Fiducial_1mm_Dia_2.54mm_Outer_CopperTop, Fiducials:Fiducial_1mm_Dia_2.54mm_Outer_CopperTop, F.Cu at (337.5, 200.0)
- added REF**: Fiducial_1mm_Dia_2.54mm_Outer_CopperTop, Fiducials:Fiducial_1mm_Dia_2.54mm_Outer_CopperTop, F.Cu at (89.5, 200.0)
- added U24: INA219AIDCNR, project:Texas_Instruments-DCN0008A-0-0-MFG, F.Cu at (226.5, 200.5)
- moved C4 6.84 mm to (219.7, 189.3), turned to 90 degrees
Connections:
- J1 pad 1: +5VP -> /VIN
Routing:
- net +5VP: track 930.4 -> 1714.4 mm, vias 50 -> 20
- net /IRQP: track 2.05 -> 292.9 mm, vias 0 -> 30
- net /SCLP: track 121.7 -> 378.2 mm, vias 0 -> 30
- net /SDAP: track 142.7 -> 380.4 mm, vias 20 -> 30
- net /CLK2: track 9.92 -> 241.4 mm, vias 0 -> 13
- net /CLK3: track 9.92 -> 237.7 mm, vias 0 -> 13
- net /CLK1: track 9.92 -> 234.7 mm, vias 0 -> 13
- net GND: track 1063.3 -> 860.5 mm, vias 164 -> 226
- net /RXP: track 2.05 -> 120.8 mm, vias 0 -> 2
- net /TXP: track 2.05 -> 110.5 mm, vias 0 -> 2
- net /CLK5: track 9.92 -> 101.0 mm, vias 0 -> 8
- net /CLK4: track 9.92 -> 96.5 mm, vias 0 -> 8
- net /TX: track 97.1 -> 28.1 mm, vias 6 -> 2
- net /IRQ: track 92.5 -> 24.4 mm, vias 4 -> 1
- net /SDA: track 125.3 -> 155.0 mm, vias 6 -> 8
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
Commit message: route complete
Routing:
- net /SDAP: track 380.4 -> 541.0 mm, vias 30 -> 32
- net /SCLP: track 378.2 -> 532.1 mm, vias 30 -> 32
- net /CLK5: track 101.0 -> 247.2 mm, vias 8 -> 12
- net /IRQP: track 292.9 -> 435.2 mm, vias 30 -> 32
- net /CLK4: track 96.5 -> 234.0 mm, vias 8 -> 10
- net /IRQ: track 24.4 -> 96.0 mm, vias 1 -> 8
- net /TX: track 28.1 -> 89.4 mm, vias 2 -> 6
- net /SDA: track 155.0 -> 133.3 mm, vias 8 -> 9
- net /CLK3: track 237.7 -> 251.6 mm, vias 13 -> 14
- net /CLK2: track 241.4 -> 252.5 mm, vias 13 -> 14
- net +5V: track 276.6 -> 286.1 mm, vias 7 -> 3
- net /SSEN: track 92.4 -> 101.3 mm
- net +5VP: track 1714.4 -> 1722.4 mm, vias 20 -> 24
- net /OEB: track 96.8 -> 104.2 mm
- net /SCL: track 144.2 -> 138.0 mm, vias 8 -> 4
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