File: NFCPower10.kicad_pcb (KiCad board)
At the start: 2 copper layers, 270 x 125 mm, 610 parts, among them J1 PJ-002AH, J10 SSW-102-01-T-S, J11 SSW-102-01-T-S, J12 Conn_02x03_Odd_Even, J13 SSW-102-01-T-S, J14 SSW-102-01-T-S, J15 Conn_02x03_Odd_Even, J16 SSW-102-01-T-S, J17 SSW-102-01-T-S, J18 Conn_02x03_Odd_Even, J19 SSW-102-01-T-S, J2 475890001, J20 SSW-102-01-T-S, J21 Conn_02x03_Odd_Even, J22 SSW-102-01-T-S, J23 SSW-102-01-T-S, J24 Conn_02x03_Odd_Even, J25 SSW-102-01-T-S, J26 SSW-102-01-T-S, J27 Conn_02x03_Odd_Even, J28 SSW-102-01-T-S, J29 SSW-102-01-T-S, J3 Conn_02x03_Odd_Even, J30 Conn_02x03_Odd_Even, J31 SSW-102-01-T-S, J32 SSW-102-01-T-S, J33 Conn_02x03_Odd_Even, J34 SSW-102-01-T-S, J35 SSW-102-01-T-S, J4 SSW-104-01-T-S, J5 SSW-106-02-T-S, J6 Conn_02x03_Odd_Even, J7 SSW-102-01-T-S, J8 SSW-102-01-T-S, J9 Conn_02x03_Odd_Even, Q1 BSS138, Q2 BSS138, Q3 BSS138, Q4 BSS138, Q5 BSS138, SW1 FSM2JSMAA, SW2 FSM2JSMAA, U1 ATMEGA328P-MU, U10 ATMEGA328P-MU, U11 ST25R3916-AQWT, U12 ATMEGA328P-MU, U13 ST25R3916-AQWT, U14 ATMEGA328P-MU, U15 ST25R3916-AQWT, U16 ATMEGA328P-MU, U17 ST25R3916-AQWT, U18 ATMEGA328P-MU, U19 ST25R3916-AQWT, U2 FT231XQ-R, U20 ATMEGA328P-MU, U21 ST25R3916-AQWT, U22 ATMEGA328P-MU, U23 ST25R3916-AQWT, U24 INA219AIDCNR, U3 Si5351A-B-GM, U4 ATMEGA328P-MU, U5 ST25R3916-AQWT, U6 ATMEGA328P-MU, U7 ST25R3916-AQWT, U8 ATMEGA328P-MU, U9 ST25R3916-AQWT, Y1 TSX-3225_16.0000MF09Z-AC3, Y10 Coil_49_18_6T_2Layer, Y11 Field_Sensor_54_22, Y12 TSX-3225_16.0000MF09Z-AC3, Y13 Coil_49_18_6T_2Layer, Y14 Field_Sensor_54_22, Y15 TSX-3225_16.0000MF09Z-AC3, Y16 Coil_49_18_6T_2Layer, Y17 Field_Sensor_54_22, Y18 TSX-3225_16.0000MF09Z-AC3, Y19 Coil_49_18_6T_2Layer, Y2 ABM8G-25.000MHz-B4Y-T, Y20 Field_Sensor_54_22, Y21 TSX-3225_16.0000MF09Z-AC3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

Commit message: rev 2
Parts:
- removed C121, C283, C59: CC0603KRX7R9BB102, project:YAGEO-CC0603-0-0-0
- removed C128, C245, C252, C276: CC0603KRX7R9BB103, project:YAGEO-CC0603-0-0-0
- removed C152, C97: CC0603KPX7R9BB104, project:YAGEO-CC0603-0-0-0
- removed C159, C183, C190, C214: CC0603MRX5R5BB225, project:YAGEO-CC0603-0-0-0
- removed C221: CGA3E2C0G1H060D080AA, project:TDK-CGA3E-0.3-0.1-0-0-IPC_A
- removed C66: CC0603KRX7R9BB181, project:YAGEO-CC0603-0-0-0
- removed C90: C0603C209C5GACTU, project:KEMET-C0603C-CF-0-0-MFG
- removed D13, D37, D44: BAS40-7-F, project:Diodes_Inc.-SOT23-01_2017-0-MFG
- removed D16, D58: LTST-C190KRKT, project:Lite-On-LTST-C190KRKT-MFG
- removed D23, D65: LTST-C190KGKT, project:Lite-On-LTST-C190KGKT-MFG
- removed D30: LTST-C190TBKT, project:Vishay_Lite-On-LTST-C190TBKT-Manufacturer_Recommended
- removed D51: LTST-C190KSKT, project:Lite-On-LTST-C190KSKT-MFG
- removed R104, R117, R39, R52, R60, R73: RC0603FR-071K65L, project:Yageo-RC0603-0-0-IPC_A
- removed R112, R125, R26, R34, R47, R65, R78, R86, R91, R99: RC0603FR-0710KL, project:Yageo-RC0603-0-0-IPC_A
- removed R7: RC0603FR-07100RL, project:Yageo-RC0603-0-0-IPC_A
- added C291: CC0603KPX7R9BB104, project:YAGEO-CC0603-0-0-0, F.Cu at (108.5, 167.5)
- added C292: CC0603MRX5R5BB225, project:YAGEO-CC0603-0-0-0, F.Cu at (104.5, 156.0)
- added C293: CC0603MRX5R5BB225, project:YAGEO-CC0603-0-0-0, F.Cu at (108.5, 153.5)
- added C294: CC0603KRX7R9BB103, project:YAGEO-CC0603-0-0-0, F.Cu at (104.5, 158.0)
- added C295: CC0603KRX7R9BB103, project:YAGEO-CC0603-0-0-0, F.Cu at (108.5, 151.5)
- added C296: CC0603MRX5R5BB225, project:YAGEO-CC0603-0-0-0, F.Cu at (108.5, 145.5)
- added C297: CC0603MRX5R5BB225, project:YAGEO-CC0603-0-0-0, F.Cu at (104.5, 144.5)
- added C298: CC0603KRX7R9BB103, project:YAGEO-CC0603-0-0-0, F.Cu at (108.5, 143.5)
- added C299: CC0603KRX7R9BB103, project:YAGEO-CC0603-0-0-0, F.Cu at (104.5, 142.5)
- added C300: CC0603MRX5R5BB225, project:YAGEO-CC0603-0-0-0, F.Cu at (101.5, 144.5)
- added C301: CGA3E2C0G1H060D080AA, project:TDK-CGA3E-0.3-0.1-0-0-IPC_A, F.Cu at (90.1, 167.5)
- added C302: CC0603KRX7R9BB103, project:YAGEO-CC0603-0-0-0, F.Cu at (101.5, 142.5)
- added C303: CGA3E2C0G1H060D080AA, project:TDK-CGA3E-0.3-0.1-0-0-IPC_A, F.Cu at (108.5, 147.5)
- added C304: CC0603KRX7R7BB105, project:YAGEO-CC0603-0-0-0, F.Cu at (107.8, 161.4)
- added C305: CGA3E2C0G1H060D080AA, project:TDK-CGA3E-0.3-0.1-0-0-IPC_A, F.Cu at (108.5, 149.5)
- added C306: CGA3E2C0G1H060D080AA, project:TDK-CGA3E-0.3-0.1-0-0-IPC_A, F.Cu at (96.5, 167.5)
- added C308: CC0603KRX7R6BB224, project:YAGEO-CC0603-0-0-0, F.Cu at (93.0, 160.0)
- added C309: CC0603KRX7R7BB105, project:YAGEO-CC0603-0-0-0, F.Cu at (108.5, 165.5)
- added C310: CC0603KRX7R9BB102, project:YAGEO-CC0603-0-0-0, F.Cu at (93.0, 154.0)
- added C311: CC0603KRX7R9BB102, project:YAGEO-CC0603-0-0-0, F.Cu at (108.5, 159.5)
- added C312: CC0603MRX5R5BB225, project:YAGEO-CC0603-0-0-0, F.Cu at (97.5, 158.0)
- added C313: CC0603KRX7R9BB103, project:YAGEO-CC0603-0-0-0, F.Cu at (97.5, 156.0)
- added C315: C0603C209C5GACTU, project:KEMET-C0603C-CF-0-0-MFG, F.Cu at (90.9, 141.0)
- added C316: C0603C209C5GACTU, project:KEMET-C0603C-CF-0-0-MFG, F.Cu at (110.0, 138.5)
- added C317: CC0603KRX7R9BB102, project:YAGEO-CC0603-0-0-0, F.Cu at (99.8, 139.5)
- added C318: CC0603KRX7R9BB102, project:YAGEO-CC0603-0-0-0, F.Cu at (102.5, 139.5)
- added C319: CC0603KRX7R9BB181, project:YAGEO-CC0603-0-0-0, F.Cu at (97.0, 139.0)
- added C320: CC0603MRX5R5BB225, project:YAGEO-CC0603-0-0-0, F.Cu at (116.5, 200.0)
- added C321: CC0603KPX7R9BB104, project:YAGEO-CC0603-0-0-0, F.Cu at (338.5, 92.0)
- added C322: CC0603KPX7R9BB104, project:YAGEO-CC0603-0-0-0, F.Cu at (88.5, 92.0)
- added C324: CC0603MRX5R5BB225, project:YAGEO-CC0603-0-0-0, F.Cu at (338.5, 94.0)
- added C325: CC0603MRX5R5BB225, project:YAGEO-CC0603-0-0-0, F.Cu at (88.5, 94.0)
- added C327: CC0603KPX7R9BB104, project:YAGEO-CC0603-0-0-0, F.Cu at (123.5, 201.0)
- added C328: CC0603MRX5R5BB225, project:YAGEO-CC0603-0-0-0, F.Cu at (123.5, 199.0)
- added C329: CC0603MRX5R5BB225, project:YAGEO-CC0603-0-0-0, F.Cu at (299.5, 200.0)
- added C330: CC0603KPX7R9BB104, project:YAGEO-CC0603-0-0-0, F.Cu at (306.5, 201.0)
- added C331: CC0603MRX5R5BB225, project:YAGEO-CC0603-0-0-0, F.Cu at (306.5, 199.0)
- added D67: LTST-C190KRKT, project:Lite-On-LTST-C190KRKT-MFG, F.Cu at (126.0, 171.0)
- added D68: LTST-C190KGKT, project:Lite-On-LTST-C190KGKT-MFG, F.Cu at (126.0, 174.0)
- added D69: LTST-C190TBKT, project:Vishay_Lite-On-LTST-C190TBKT-Manufacturer_Recommended, F.Cu at (126.0, 177.0)
- added D70: BAS40-7-F, project:Diodes_Inc.-SOT23-01_2017-0-MFG, F.Cu at (93.0, 151.5)
- added D71: BAS40-7-F, project:Diodes_Inc.-SOT23-01_2017-0-MFG, F.Cu at (108.5, 157.0)
- added D73: LTST-C190KSKT, project:Lite-On-LTST-C190KSKT-MFG, F.Cu at (93.0, 145.5)
- added D74: LTST-C190KRKT, project:Lite-On-LTST-C190KRKT-MFG, F.Cu at (101.0, 171.0)
- added D75: LTST-C190KGKT, project:Lite-On-LTST-C190KGKT-MFG, F.Cu at (101.0, 174.0)
- added D76: LTST-C190TBKT, project:Vishay_Lite-On-LTST-C190TBKT-Manufacturer_Recommended, F.Cu at (101.0, 177.0)
- added D77: LTST-C190KGKT, project:Lite-On-LTST-C190KGKT-MFG, B.Cu at (338.5, 85.0)
- added D78: LTST-C190KGKT, project:Lite-On-LTST-C190KGKT-MFG, B.Cu at (88.5, 85.0)
- added J36: SSW-102-01-T-S, project:Samtec-SSW-102-01-T-S-Manufacturer_Recommended, F.Cu at (101.0, 96.0)
- added J37: Conn_02x03_Odd_Even, Pin_Headers:Pin_Header_Straight_2x03_Pitch2.54mm, F.Cu at (107.5, 188.0)
- added J38: SSW-104-01-T-S, project:Samtec-SSW-104-01-T-S-Manufacturer_Recommended, F.Cu at (95.5, 188.0)
- added J39: SSW-104-01-T-S, project:Samtec-SSW-104-01-T-S-Manufacturer_Recommended, F.Cu at (101.5, 188.0)
- added Q10: BSS138, project:ON_Semiconductor-318-08-01_2018-AS-MFG, F.Cu at (332.5, 190.0)
- added Q12: BSS138, project:ON_Semiconductor-318-08-01_2018-AS-MFG, F.Cu at (338.5, 99.0)
- added Q13: BSS138, project:ON_Semiconductor-318-08-01_2018-AS-MFG, F.Cu at (88.5, 99.0)
- added Q15: BSS138, project:ON_Semiconductor-318-08-01_2018-AS-MFG, F.Cu at (129.5, 188.0)
- added Q16: BSS138, project:ON_Semiconductor-318-08-01_2018-AS-MFG, F.Cu at (123.5, 188.0)
- added Q17: BSS138, project:ON_Semiconductor-318-08-01_2018-AS-MFG, F.Cu at (117.5, 193.0)
- added Q18: BSS138, project:ON_Semiconductor-318-08-01_2018-AS-MFG, F.Cu at (135.5, 188.0)
- added Q19: BSS138, project:ON_Semiconductor-318-08-01_2018-AS-MFG, F.Cu at (117.5, 188.0)
- added Q20: BSS138, project:ON_Semiconductor-318-08-01_2018-AS-MFG, F.Cu at (123.5, 193.0)
- added Q6: BSS138, project:ON_Semiconductor-318-08-01_2018-AS-MFG, F.Cu at (317.5, 195.0)
- added Q7: BSS138, project:ON_Semiconductor-318-08-01_2018-AS-MFG, F.Cu at (317.5, 190.0)
- added Q8: BSS138, project:ON_Semiconductor-318-08-01_2018-AS-MFG, F.Cu at (326.5, 195.0)
- added Q9: BSS138, project:ON_Semiconductor-318-08-01_2018-AS-MFG, F.Cu at (326.5, 190.0)
- added R131: RC0603FR-071K65L, project:Yageo-RC0603-0-0-IPC_A, F.Cu at (118.0, 147.5)
- added R132: RC0603FR-071K65L, project:Yageo-RC0603-0-0-IPC_A, F.Cu at (122.0, 171.0)
- added R133: RC0603FR-071K65L, project:Yageo-RC0603-0-0-IPC_A, F.Cu at (122.0, 174.0)
- added R134: RC0603FR-071K65L, project:Yageo-RC0603-0-0-IPC_A, F.Cu at (122.0, 177.0)
- added R135: RC0603FR-0710KL, project:Yageo-RC0603-0-0-IPC_A, F.Cu at (101.0, 156.0)
- added R136: RC0603FR-0710KL, project:Yageo-RC0603-0-0-IPC_A, F.Cu at (101.0, 158.0)
- added R137: RC0603FR-071K65L, project:Yageo-RC0603-0-0-IPC_A, F.Cu at (106.4, 138.5)
- added R139: RC0603FR-0710KL, project:Yageo-RC0603-0-0-IPC_A, F.Cu at (90.5, 176.0)
- added R140: RC0603FR-0710KL, project:Yageo-RC0603-0-0-IPC_A, F.Cu at (93.0, 156.0)
- added R141: RC0603FR-071K65L, project:Yageo-RC0603-0-0-IPC_A, F.Cu at (108.5, 163.4)
- added R142: RC0603FR-0710KL, project:Yageo-RC0603-0-0-IPC_A, F.Cu at (93.0, 158.0)
- added R144: RC0603FR-071K65L, project:Yageo-RC0603-0-0-IPC_A, F.Cu at (93.0, 147.5)
- added R145: RC0603FR-071K65L, project:Yageo-RC0603-0-0-IPC_A, F.Cu at (97.0, 171.0)
- added R146: RC0603FR-071K65L, project:Yageo-RC0603-0-0-IPC_A, F.Cu at (97.0, 174.0)
- added R147: RC0603FR-071K65L, project:Yageo-RC0603-0-0-IPC_A, F.Cu at (97.0, 177.0)
- added R148: RC0603FR-0710KL, project:Yageo-RC0603-0-0-IPC_A, F.Cu at (320.5, 190.0)
- added R149: RC0603FR-071K65L, project:Yageo-RC0603-0-0-IPC_A, F.Cu at (314.5, 195.0)
- added R150: RC0603FR-0710KL, project:Yageo-RC0603-0-0-IPC_A, F.Cu at (314.5, 190.0)
- added R151: RC0603FR-071K65L, project:Yageo-RC0603-0-0-IPC_A, F.Cu at (323.5, 195.0)
- added R152: RC0603FR-0710KL, project:Yageo-RC0603-0-0-IPC_A, F.Cu at (323.5, 190.0)
- added R153: RC0603FR-0710KL, project:Yageo-RC0603-0-0-IPC_A, F.Cu at (329.5, 190.0)
- added R154: RC0603FR-071K65L, project:Yageo-RC0603-0-0-IPC_A, F.Cu at (338.5, 96.0)
- added R155: RC0603FR-071K65L, project:Yageo-RC0603-0-0-IPC_A, F.Cu at (88.5, 96.0)
- added R158: RC0603FR-071K65L, project:Yageo-RC0603-0-0-IPC_A, F.Cu at (126.5, 188.0)
- added R159: RC0603FR-071K65L, project:Yageo-RC0603-0-0-IPC_A, F.Cu at (120.5, 188.0)
- added R160: RC0603FR-071K65L, project:Yageo-RC0603-0-0-IPC_A, F.Cu at (114.5, 193.0)
- added R161: RC0603FR-071K65L, project:Yageo-RC0603-0-0-IPC_A, F.Cu at (132.5, 188.0)
- added R162: RC0603FR-071K65L, project:Yageo-RC0603-0-0-IPC_A, F.Cu at (114.5, 188.0)
- added R163: RC0603FR-071K65L, project:Yageo-RC0603-0-0-IPC_A, F.Cu at (120.5, 193.0)
- added U25: LP3985IM5X-2.8_NOPB, project:TI_National_Semiconductor-LP3985IM5X-2.8_NOPB-Level_A, F.Cu at (302.5, 200.0)
- added U26: LP3985IM5X-3.3_NOPB, project:TI_National_Semiconductor-LP3985IM5X-3.3_NOPB-Level_A, F.Cu at (119.5, 200.0)
- added UED1: VL6180XV0NR_1, project:STMicroelectronics-VL6180XV0NR_1-MFG, B.Cu at (338.5, 88.0)
- added UED2: VL6180XV0NR_1, project:STMicroelectronics-VL6180XV0NR_1-MFG, B.Cu at (88.5, 88.0)
- C100, C101, C132, C156, C217, C224, C225, C248, C280: value CC0603KRX7R9BB103 -> CC0603KRX7R9BB102
- C102, C71: value CC0603MRX5R5BB225 -> CC0603KRX7R9BB181
- C103, C134: value CC0603MRX5R5BB225 -> CC0805ZKY5V6BB106; footprint project:YAGEO-CC0603-0-0-0 -> project:YAGEO-CC0805-0-0-0
- C104, C105, C136, C197, C229, C73: value CC0603KRX7R9BB103 -> CC0603KPX7R9BB104
- C107, C110, C111, C137, C138, C219, C250, C79, C83: value CGA3E2C0G1H060D080AA -> CC0603MRX5R5BB225; footprint project:TDK-CGA3E-0.3-0.1-0-0-IPC_A -> project:YAGEO-CC0603-0-0-0
- C109, C139, C251, C51, C54, C81, C82: value CGA3E2C0G1H060D080AA -> CC0603KRX7R9BB103; footprint project:TDK-CGA3E-0.3-0.1-0-0-IPC_A -> project:YAGEO-CC0603-0-0-0
- C114, C142, C176, C199, C204, C261, C64: value CC0603KRX7R9BB102 -> CC0603MRX5R5BB225
- C115, C120, C148, C177, C58, C86: value CC0603KRX7R9BB102 -> CGA3E2C0G1H060D080AA; footprint project:YAGEO-CC0603-0-0-0 -> project:TDK-CGA3E-0.3-0.1-0-0-IPC_A
- C116, C127, C144, C158, C267, C271, C46, C47, C50, C78: value CC0603MRX5R5BB225 -> CC0603KRX7R9BB103
- C117, C212, C213, C241, C244, C272, C57, C84, C89: value CC0603KRX7R9BB103 -> CGA3E2C0G1H060D080AA; footprint project:YAGEO-CC0603-0-0-0 -> project:TDK-CGA3E-0.3-0.1-0-0-IPC_A
- C118: value C0603C209C5GACTU -> CC0603KRX7R7BB105; footprint project:KEMET-C0603C-CF-0-0-MFG -> project:YAGEO-CC0603-0-0-0
- C119, C146: value C0603C209C5GACTU -> CGA3E2C0G1H060D080AA; footprint project:KEMET-C0603C-CF-0-0-MFG -> project:TDK-CGA3E-0.3-0.1-0-0-IPC_A
- C122: value CC0603KRX7R9BB181 -> CC0603KRX7R6BB224
- C123: value CC0805ZKY5V6BB106 -> CC0603KRX7R7BB105; footprint project:YAGEO-CC0805-0-0-0 -> project:YAGEO-CC0603-0-0-0
- C124, C125, C69: value CC0603KPX7R9BB104 -> CC0603KRX7R9BB102
- C129, C160, C161, C192, C253, C285: value CC0603KRX7R9BB103 -> C0603C209C5GACTU; footprint project:YAGEO-CC0603-0-0-0 -> project:KEMET-C0603C-CF-0-0-MFG
- C130, C284, C98, C99: value CC0603MRX5R5BB225 -> C0603C209C5GACTU; footprint project:YAGEO-CC0603-0-0-0 -> project:KEMET-C0603C-CF-0-0-MFG
- C131, C155, C162, C186, C187, C218, C256, C70: value CC0603MRX5R5BB225 -> CC0603KRX7R9BB102
- C133, C164, C257: value CC0603KRX7R9BB103 -> CC0603KRX7R9BB181
- C135, C166, C167: value CGA3E2C0G1H060D080AA -> CC0603KPX7R9BB104; footprint project:TDK-CGA3E-0.3-0.1-0-0-IPC_A -> project:YAGEO-CC0603-0-0-0
- C141, C145, C157, C168, C169, C173, C188, C269, C281, C44, C45, C48, C49, C52, C76, C80: value CC0603KRX7R9BB103 -> CC0603MRX5R5BB225
- C143, C170, C171, C205, C232, C233, C282, C65: value CC0603KRX7R9BB102 -> CC0603KRX7R9BB103
- C147, C174, C175, C202: value C0603C209C5GACTU -> CC0603KRX7R9BB103; footprint project:KEMET-C0603C-CF-0-0-MFG -> project:YAGEO-CC0603-0-0-0
- C149, C87, C92: value CC0603KRX7R9BB102 -> CC0603KRX7R7BB105
- C150: value CC0603KRX7R9BB181 -> CGA3E2C0G1H060D080AA; footprint project:YAGEO-CC0603-0-0-0 -> project:TDK-CGA3E-0.3-0.1-0-0-IPC_A
- C151, C179: value CC0805ZKY5V6BB106 -> CGA3E2C0G1H060D080AA; footprint project:YAGEO-CC0805-0-0-0 -> project:TDK-CGA3E-0.3-0.1-0-0-IPC_A
- C153: value CC0603KPX7R9BB104 -> CC0603KRX7R6BB224
- C154, C211, C242: value CC0603MRX5R5BB225 -> CC0603KRX7R7BB105
- C163, C193, C194, C249, C279: value CGA3E2C0G1H060D080AA -> CC0603KRX7R9BB102; footprint project:TDK-CGA3E-0.3-0.1-0-0-IPC_A -> project:YAGEO-CC0603-0-0-0
- C165: value CGA3E2C0G1H060D080AA -> CC0805ZKY5V6BB106; footprint project:TDK-CGA3E-0.3-0.1-0-0-IPC_A -> project:YAGEO-CC0805-0-0-0
- C178, C206: value CC0603KRX7R9BB181 -> CC0603KRX7R9BB103
- C180, C40: value CC0603KPX7R9BB104 -> CC0603KRX7R7BB105
- C181, C208: value CC0603KPX7R9BB104 -> CGA3E2C0G1H060D080AA; footprint project:YAGEO-CC0603-0-0-0 -> project:TDK-CGA3E-0.3-0.1-0-0-IPC_A
- C182, C210, C239, C243, C270, C274, C88: value CC0603MRX5R5BB225 -> CGA3E2C0G1H060D080AA; footprint project:YAGEO-CC0603-0-0-0 -> project:TDK-CGA3E-0.3-0.1-0-0-IPC_A
- C184, C28: value CC0603KRX7R9BB103 -> CC0603KRX7R6BB224
- C185, C216, C273, C29, C56, C61: value CC0603KRX7R9BB103 -> CC0603KRX7R7BB105
- C191, C222, C223: value CGA3E2C0G1H060D080AA -> C0603C209C5GACTU; footprint project:TDK-CGA3E-0.3-0.1-0-0-IPC_A -> project:KEMET-C0603C-CF-0-0-MFG
- C195: value CGA3E2C0G1H060D080AA -> CC0603KRX7R9BB181; footprint project:TDK-CGA3E-0.3-0.1-0-0-IPC_A -> project:YAGEO-CC0603-0-0-0
- C196, C72: value CC0603KRX7R9BB103 -> CC0805ZKY5V6BB106; footprint project:YAGEO-CC0603-0-0-0 -> project:YAGEO-CC0805-0-0-0
- C198, C260: value CC0603KRX7R9BB102 -> CC0603KPX7R9BB104
- C203, C230, C231: value C0603C209C5GACTU -> CC0603MRX5R5BB225; footprint project:KEMET-C0603C-CF-0-0-MFG -> project:YAGEO-CC0603-0-0-0
- C207, C235, C95: value CC0805ZKY5V6BB106 -> CC0603MRX5R5BB225; footprint project:YAGEO-CC0805-0-0-0 -> project:YAGEO-CC0603-0-0-0
- C209, C236, C237, C264, C96: value CC0603KPX7R9BB104 -> CC0603KRX7R9BB103
- C215, C246, C60: value CC0603MRX5R5BB225 -> CC0603KRX7R6BB224
- C226, C288: value CC0603KRX7R9BB102 -> CC0603KRX7R9BB181
- C227, C289: value CC0603KRX7R9BB102 -> CC0805ZKY5V6BB106; footprint project:YAGEO-CC0603-0-0-0 -> project:YAGEO-CC0805-0-0-0
- C228, C42, C43, C74: value CC0603MRX5R5BB225 -> CC0603KPX7R9BB104
- C234, C262: value CC0603KRX7R9BB181 -> CC0603MRX5R5BB225
- C247, C278: value CGA3E2C0G1H060D080AA -> CC0603KRX7R7BB105; footprint project:TDK-CGA3E-0.3-0.1-0-0-IPC_A -> project:YAGEO-CC0603-0-0-0
- C254: value CC0603KRX7R9BB102 -> C0603C209C5GACTU; footprint project:YAGEO-CC0603-0-0-0 -> project:KEMET-C0603C-CF-0-0-MFG
- C258: value C0603C209C5GACTU -> CC0805ZKY5V6BB106; footprint project:KEMET-C0603C-CF-0-0-MFG -> project:YAGEO-CC0805-0-0-0
- C259: value C0603C209C5GACTU -> CC0603KPX7R9BB104; footprint project:KEMET-C0603C-CF-0-0-MFG -> project:YAGEO-CC0603-0-0-0
- C263: value CC0805ZKY5V6BB106 -> CC0603KRX7R9BB103; footprint project:YAGEO-CC0805-0-0-0 -> project:YAGEO-CC0603-0-0-0
- C265: value CC0603KPX7R9BB104 -> CC0603MRX5R5BB225
- C277: value CGA3E2C0G1H060D080AA -> CC0603KRX7R6BB224; footprint project:TDK-CGA3E-0.3-0.1-0-0-IPC_A -> project:YAGEO-CC0603-0-0-0
- C286, C287, C62, C63: value C0603C209C5GACTU -> CC0603KRX7R9BB102; footprint project:KEMET-C0603C-CF-0-0-MFG -> project:YAGEO-CC0603-0-0-0
- C290: value CC0603KRX7R9BB181 -> CC0603KPX7R9BB104
- C39: value CC0805ZKY5V6BB106 -> CC0603KPX7R9BB104; footprint project:YAGEO-CC0805-0-0-0 -> project:YAGEO-CC0603-0-0-0
- C41: value CC0603KPX7R9BB104 -> CC0805ZKY5V6BB106; footprint project:YAGEO-CC0603-0-0-0 -> project:YAGEO-CC0805-0-0-0
- C67: value CC0805ZKY5V6BB106 -> C0603C209C5GACTU; footprint project:YAGEO-CC0805-0-0-0 -> project:KEMET-C0603C-CF-0-0-MFG
- C68: value CC0603KPX7R9BB104 -> C0603C209C5GACTU; footprint project:YAGEO-CC0603-0-0-0 -> project:KEMET-C0603C-CF-0-0-MFG
- C91: value C0603C209C5GACTU -> CC0603KRX7R6BB224; footprint project:KEMET-C0603C-CF-0-0-MFG -> project:YAGEO-CC0603-0-0-0
- C94: value CC0603KRX7R9BB181 -> CC0603KRX7R9BB102
- D15, D21, D57, D63: value LTST-C190KSKT -> BAS40-7-F; footprint project:Lite-On-LTST-C190KSKT-MFG -> project:Diodes_Inc.-SOT23-01_2017-0-MFG
- D17, D59: value LTST-C190KGKT -> LTST-C190KSKT; footprint project:Lite-On-LTST-C190KGKT-MFG -> project:Lite-On-LTST-C190KSKT-MFG
- D18, D60: value LTST-C190TBKT -> LTST-C190KRKT; footprint project:Vishay_Lite-On-LTST-C190TBKT-Manufacturer_Recommended -> project:Lite-On-LTST-C190KRKT-MFG
- D19, D26, D61: value BAS40-7-F -> LTST-C190KGKT; footprint project:Diodes_Inc.-SOT23-01_2017-0-MFG -> project:Lite-On-LTST-C190KGKT-MFG
- D20, D55, D62: value BAS40-7-F -> LTST-C190TBKT; footprint project:Diodes_Inc.-SOT23-01_2017-0-MFG -> project:Vishay_Lite-On-LTST-C190TBKT-Manufacturer_Recommended
- D22, D28, D64: value LTST-C190KRKT -> BAS40-7-F; footprint project:Lite-On-LTST-C190KRKT-MFG -> project:Diodes_Inc.-SOT23-01_2017-0-MFG
- D24, D66: value LTST-C190TBKT -> LTST-C190KSKT; footprint project:Vishay_Lite-On-LTST-C190TBKT-Manufacturer_Recommended -> project:Lite-On-LTST-C190KSKT-MFG
- D25, D32: value BAS40-7-F -> LTST-C190KRKT; footprint project:Diodes_Inc.-SOT23-01_2017-0-MFG -> project:Lite-On-LTST-C190KRKT-MFG
- D27: value LTST-C190KSKT -> LTST-C190TBKT; footprint project:Lite-On-LTST-C190KSKT-MFG -> project:Vishay_Lite-On-LTST-C190TBKT-Manufacturer_Recommended
- D29, D35: value LTST-C190KGKT -> BAS40-7-F; footprint project:Lite-On-LTST-C190KGKT-MFG -> project:Diodes_Inc.-SOT23-01_2017-0-MFG
- D31, D38: value BAS40-7-F -> LTST-C190KSKT; footprint project:Diodes_Inc.-SOT23-01_2017-0-MFG -> project:Lite-On-LTST-C190KSKT-MFG
- D33: value LTST-C190KSKT -> LTST-C190KGKT; footprint project:Lite-On-LTST-C190KSKT-MFG -> project:Lite-On-LTST-C190KGKT-MFG
- D34: value LTST-C190KRKT -> LTST-C190TBKT; footprint project:Lite-On-LTST-C190KRKT-MFG -> project:Vishay_Lite-On-LTST-C190TBKT-Manufacturer_Recommended
- D36, D42: value LTST-C190TBKT -> BAS40-7-F; footprint project:Vishay_Lite-On-LTST-C190TBKT-Manufacturer_Recommended -> project:Diodes_Inc.-SOT23-01_2017-0-MFG
- D39: value LTST-C190KSKT -> LTST-C190KRKT; footprint project:Lite-On-LTST-C190KSKT-MFG -> project:Lite-On-LTST-C190KRKT-MFG
- D40: value LTST-C190KRKT -> LTST-C190KGKT; footprint project:Lite-On-LTST-C190KRKT-MFG -> project:Lite-On-LTST-C190KGKT-MFG
- D41: value LTST-C190KGKT -> LTST-C190TBKT; footprint project:Lite-On-LTST-C190KGKT-MFG -> project:Vishay_Lite-On-LTST-C190TBKT-Manufacturer_Recommended
- D52: value LTST-C190KRKT -> LTST-C190KSKT; footprint project:Lite-On-LTST-C190KRKT-MFG -> project:Lite-On-LTST-C190KSKT-MFG
- D53: value LTST-C190KGKT -> LTST-C190KRKT; footprint project:Lite-On-LTST-C190KGKT-MFG -> project:Lite-On-LTST-C190KRKT-MFG
- D54: value LTST-C190TBKT -> LTST-C190KGKT; footprint project:Vishay_Lite-On-LTST-C190TBKT-Manufacturer_Recommended -> project:Lite-On-LTST-C190KGKT-MFG
- FID1, FID2, FID3: renamed from REF**; value Fiducial_1mm_Dia_2.54mm_Outer_CopperTop -> fiducial
- J10, J13, J16, J19, J22, J25, J28, J31, J34: value SSW-102-01-T-S -> Conn_02x03_Odd_Even; footprint project:Samtec-SSW-102-01-T-S-Manufacturer_Recommended -> Pin_Headers:Pin_Header_Straight_2x03_Pitch2.54mm
- J11, J14, J17, J20, J23, J26, J29, J32, J35, J7: value SSW-102-01-T-S -> SSW-104-01-T-S; footprint project:Samtec-SSW-102-01-T-S-Manufacturer_Recommended -> project:Samtec-SSW-104-01-T-S-Manufacturer_Recommended
- J12, J15, J18, J21, J24, J27, J30, J33: value Conn_02x03_Odd_Even -> SSW-102-01-T-S; footprint Pin_Headers:Pin_Header_Straight_2x03_Pitch2.54mm -> project:Samtec-SSW-102-01-T-S-Manufacturer_Recommended
- J9: value Conn_02x03_Odd_Even -> SSW-104-01-T-S; footprint Pin_Headers:Pin_Header_Straight_2x03_Pitch2.54mm -> project:Samtec-SSW-104-01-T-S-Manufacturer_Recommended
- MT1, MT2, MT3, MT4: renamed from REF**; value MountingHole_3.2mm_M3 -> Mount Hole M3
- R102, R108, R11, R111, R119, R12, R120, R121, R124, R24, R33, R37, R42, R43, R46, R53, R54, R55, R56, R59, R66, R67, R68, R69, R76, R79, R80, R81, R89, R92, R98: value RC0603FR-0710KL -> RC0603FR-071K65L
- R116, R126, R127, R129, R38, R49, R51, R61, R62, R71, R74, R83, R84, R96: value RC0603FR-071K65L -> RC0603FR-0710KL
- R6: value RC0603FR-07100RL -> RC0603FR-071K65L
- Y10, Y13, Y16, Y19, Y22, Y25, Y28, Y31, Y7: value Coil_49_18_6T_2Layer -> Field_Sensor_54_22; footprint project:Coil_49_18_6T_2Layer -> project:Field_Sensor_54_22; moved to B.Cu
- Y11, Y14, Y17, Y20, Y23, Y26, Y29, Y32, Y8: value Field_Sensor_54_22 -> TSX-3225_16.0000MF09Z-AC3; footprint project:Field_Sensor_54_22 -> project:Epson-TSX-3225_16.0000MF09Z-AC3-0; moved to F.Cu
- Y12, Y15, Y18, Y21, Y24, Y27, Y30, Y6, Y9: value TSX-3225_16.0000MF09Z-AC3 -> Coil_49_18_6T_2Layer; footprint project:Epson-TSX-3225_16.0000MF09Z-AC3-0 -> project:Coil_49_18_6T_2Layer
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Connections:
- net /CS renamed /SDCS
- C10 pad 1: +5V -> /DEV1/3V3
- C100 pad 1: +5VP -> /TX3/RF2
- C101 pad 1: /TX4/VDD_D -> GND
- C101 pad 2: GND -> /TX3/RF1
- C102 pad 1: /TX4/VDD_A -> /TX3/RF2
- C102 pad 2: GND -> Net-(C102-Pad2)
- C103 pad 1: /TX4/VDD_RF -> GND
- C103 pad 2: GND -> +5VP
- C104 pad 1: /TX4/VDD_A -> +5VP
- C105 pad 1: /TX4/VDD_RF -> Net-(C105-Pad1)
- C106 pad 1: /TX4/VDD_AM -> +5VP
- C107 pad 1: Net-(C107-Pad1) -> /TX4/VDD_D
- C108 pad 1: /TX4/VDD_AM -> +5VP
- C109 pad 1: /CLK4 -> /TX4/VDD_D
- C110 pad 1: Net-(C110-Pad1) -> /TX4/VDD_A
- C111 pad 1: Net-(C111-Pad1) -> /TX4/VDD_RF
- C112 pad 1: /TX4/VDET1 -> /TX4/VDD_A
- C113 pad 1: /TX4/VDET2 -> /TX4/VDD_RF
- C114 pad 1: Net-(C114-Pad1) -> /TX4/VDD_AM
- C116 pad 1: /TX4/AGDC -> /TX4/VDD_AM
- C117 pad 1: /TX4/AGDC -> /CLK4
- C118 pad 1: /TX4/HSEN1 -> /TX4/VPD2
- C119 pad 1: /TX4/HSEN2 -> Net-(C119-Pad1)
- C120 pad 1: /TX4/RF2 -> Net-(C120-Pad1)
- C122 pad 1: /TX4/RF2 -> /TX4/VDET1
- C122 pad 2: Net-(C122-Pad2) -> GND
- C123 pad 1: GND -> /TX4/VDET2
- C123 pad 2: +5VP -> GND
- C124 pad 1: +5VP -> Net-(C124-Pad1)
- C126 pad 1: +5VP -> /TX4/AGDC
- C127 pad 1: /TX5/VDD_D -> /TX4/AGDC
- C129 pad 1: /TX5/VDD_D -> /TX4/HSEN1
- C130 pad 1: /TX5/VDD_A -> /TX4/HSEN2
- C131 pad 1: /TX5/VDD_RF -> /TX4/RF2
- C132 pad 1: /TX5/VDD_A -> GND
- C132 pad 2: GND -> /TX4/RF1
- C133 pad 1: /TX5/VDD_RF -> /TX4/RF2
- C133 pad 2: GND -> Net-(C133-Pad2)
- C134 pad 1: /TX5/VDD_AM -> GND
- C134 pad 2: GND -> +5VP
- C135 pad 1: Net-(C135-Pad1) -> +5VP
- C136 pad 1: /TX5/VDD_AM -> Net-(C136-Pad1)
- C137 pad 1: /CLK5 -> +5VP
- C138 pad 1: Net-(C138-Pad1) -> /TX5/VDD_D
- C139 pad 1: Net-(C139-Pad1) -> +5VP
- C140 pad 1: /TX5/VDET1 -> /TX5/VDD_D
- C141 pad 1: /TX5/VDET2 -> /TX5/VDD_A
- C142 pad 1: Net-(C142-Pad1) -> /TX5/VDD_RF
- C143 pad 1: Net-(C143-Pad1) -> /TX5/VDD_A
- C144 pad 1: /TX5/AGDC -> /TX5/VDD_RF
- C145 pad 1: /TX5/AGDC -> /TX5/VDD_AM
- C146 pad 1: /TX5/HSEN1 -> Net-(C146-Pad1)
- C147 pad 1: /TX5/HSEN2 -> /TX5/VDD_AM
- C148 pad 1: /TX5/RF2 -> /CLK5
- C149 pad 1: GND -> /TX5/VPD2
- C149 pad 2: /TX5/RF1 -> GND
- C150 pad 1: /TX5/RF2 -> Net-(C150-Pad1)
- C150 pad 2: Net-(C150-Pad2) -> GND
- C151 pad 1: GND -> Net-(C151-Pad1)
- C151 pad 2: +5VP -> GND
- C153 pad 1: Net-(C153-Pad1) -> /TX5/VDET1
- C154 pad 1: +5VP -> /TX5/VDET2
- C155 pad 1: /TX6/VDD_D -> Net-(C155-Pad1)
- C156 pad 1: +5VP -> Net-(C156-Pad1)
- C157 pad 1: /TX6/VDD_D -> /TX5/AGDC
- C158 pad 1: /TX6/VDD_A -> /TX5/AGDC
- C160 pad 1: /TX6/VDD_A -> /TX5/HSEN1
- C161 pad 1: /TX6/VDD_RF -> /TX5/HSEN2
- C162 pad 1: /TX6/VDD_AM -> /TX5/RF2
- C163 pad 1: Net-(C163-Pad1) -> GND
- C163 pad 2: GND -> /TX5/RF1
- C164 pad 1: /TX6/VDD_AM -> /TX5/RF2
- C164 pad 2: GND -> Net-(C164-Pad2)
- C165 pad 1: /CLK1 -> GND
- C165 pad 2: GND -> +5VP
- C166 pad 1: Net-(C166-Pad1) -> +5VP
- C168 pad 1: /TX6/VDET1 -> +5VP
- C169 pad 1: /TX6/VDET2 -> /TX6/VDD_D
- C170 pad 1: Net-(C170-Pad1) -> +5VP
- C171 pad 1: Net-(C171-Pad1) -> /TX6/VDD_D
- C172 pad 1: /TX6/AGDC -> /TX6/VDD_A
- C173 pad 1: /TX6/AGDC -> /TX6/VDD_RF
- C174 pad 1: /TX6/HSEN1 -> /TX6/VDD_A
- C175 pad 1: /TX6/HSEN2 -> /TX6/VDD_RF
- C176 pad 1: /TX6/RF2 -> /TX6/VDD_AM
- C177 pad 1: GND -> Net-(C177-Pad1)
- C177 pad 2: /TX6/RF1 -> GND
- C178 pad 1: /TX6/RF2 -> /TX6/VDD_AM
- C178 pad 2: Net-(C178-Pad2) -> GND
- C179 pad 1: GND -> /CLK1
- C179 pad 2: +5VP -> GND
- C180 pad 1: +5VP -> /TX6/VPD2
- C182 pad 1: +5VP -> Net-(C182-Pad1)
- C184 pad 1: +5VP -> /TX6/VDET1
- C185 pad 1: /TX7/VDD_D -> /TX6/VDET2
- C186 pad 1: /TX7/VDD_A -> Net-(C186-Pad1)
- C187 pad 1: /TX7/VDD_RF -> Net-(C187-Pad1)
- C188 pad 1: /TX7/VDD_A -> /TX6/AGDC
- C189 pad 1: /TX7/VDD_RF -> /TX6/AGDC
- C191 pad 1: Net-(C191-Pad1) -> /TX6/HSEN1
- C192 pad 1: /TX7/VDD_AM -> /TX6/HSEN2
- C193 pad 1: /CLK2 -> /TX6/RF2
- C194 pad 1: Net-(C194-Pad1) -> GND
- C194 pad 2: GND -> /TX6/RF1
- C195 pad 1: Net-(C195-Pad1) -> /TX6/RF2
- C195 pad 2: GND -> Net-(C195-Pad2)
- C196 pad 1: /TX7/VDET1 -> GND
- C196 pad 2: GND -> +5VP
- C197 pad 1: /TX7/VDET2 -> +5VP
- C199 pad 1: Net-(C199-Pad1) -> +5VP
- C200 pad 1: /TX7/AGDC -> /TX7/VDD_D
- C201 pad 1: /TX7/AGDC -> +5VP
- C202 pad 1: /TX7/HSEN1 -> /TX7/VDD_D
- C203 pad 1: /TX7/HSEN2 -> /TX7/VDD_A
- C204 pad 1: /TX7/RF2 -> /TX7/VDD_RF
- C205 pad 1: GND -> /TX7/VDD_A
- C205 pad 2: /TX7/RF1 -> GND
- C206 pad 1: /TX7/RF2 -> /TX7/VDD_RF
- C206 pad 2: Net-(C206-Pad2) -> GND
- C207 pad 1: GND -> /TX7/VDD_AM
- C207 pad 2: +5VP -> GND
- C208 pad 1: +5VP -> Net-(C208-Pad1)
- C209 pad 1: Net-(C209-Pad1) -> /TX7/VDD_AM
- C210 pad 1: +5VP -> /CLK2
- C211 pad 1: /TX8/VDD_D -> /TX7/VPD2
- C212 pad 1: +5VP -> Net-(C212-Pad1)
- C213 pad 1: /TX8/VDD_D -> Net-(C213-Pad1)
- C215 pad 1: /TX8/VDD_RF -> /TX7/VDET1
- C216 pad 1: /TX8/VDD_A -> /TX7/VDET2
- C217 pad 1: /TX8/VDD_RF -> Net-(C217-Pad1)
- C218 pad 1: /TX8/VDD_AM -> Net-(C218-Pad1)
- C219 pad 1: Net-(C219-Pad1) -> /TX7/AGDC
- C220 pad 1: /TX8/VDD_AM -> /TX7/AGDC
- C222 pad 1: Net-(C222-Pad1) -> /TX7/HSEN1
- C223 pad 1: Net-(C223-Pad1) -> /TX7/HSEN2
- C224 pad 1: /TX8/VDET1 -> /TX7/RF2
- C225 pad 1: /TX8/VDET2 -> GND
- C225 pad 2: GND -> /TX7/RF1
- C226 pad 1: Net-(C226-Pad1) -> /TX7/RF2
- C226 pad 2: GND -> Net-(C226-Pad2)
- C227 pad 1: Net-(C227-Pad1) -> GND
- C227 pad 2: GND -> +5VP
- C228 pad 1: /TX8/AGDC -> +5VP
- C229 pad 1: /TX8/AGDC -> Net-(C229-Pad1)
- C230 pad 1: /TX8/HSEN1 -> +5VP
- C231 pad 1: /TX8/HSEN2 -> /TX8/VDD_D
- C232 pad 1: /TX8/RF2 -> +5VP
- C233 pad 1: GND -> /TX8/VDD_D
- C233 pad 2: /TX8/RF1 -> GND
- C234 pad 1: /TX8/RF2 -> /TX8/VDD_A
- C234 pad 2: Net-(C234-Pad2) -> GND
- C235 pad 1: GND -> /TX8/VDD_RF
- C235 pad 2: +5VP -> GND
- C236 pad 1: +5VP -> /TX8/VDD_A
- C237 pad 1: Net-(C237-Pad1) -> /TX8/VDD_RF
- C238 pad 1: +5VP -> /TX8/VDD_AM
- C239 pad 1: /TX9/VDD_D -> Net-(C239-Pad1)
- C240 pad 1: +5VP -> /TX8/VDD_AM
- C241 pad 1: /TX9/VDD_D -> /CLK3
- C242 pad 1: /TX9/VDD_A -> /TX8/VPD2
- C243 pad 1: /TX9/VDD_RF -> Net-(C243-Pad1)
- C244 pad 1: /TX9/VDD_A -> Net-(C244-Pad1)
- C246 pad 1: /TX9/VDD_AM -> /TX8/VDET1
- C247 pad 1: Net-(C247-Pad1) -> /TX8/VDET2
- C248 pad 1: /TX9/VDD_AM -> Net-(C248-Pad1)
- C249 pad 1: /CLK4 -> Net-(C249-Pad1)
- C250 pad 1: Net-(C250-Pad1) -> /TX8/AGDC
- C251 pad 1: Net-(C251-Pad1) -> /TX8/AGDC
- C253 pad 1: /TX9/VDET2 -> /TX8/HSEN1
- C254 pad 1: Net-(C254-Pad1) -> /TX8/HSEN2
- C255 pad 1: Net-(C255-Pad1) -> /TX8/RF2
- C256 pad 1: /TX9/AGDC -> GND
- C256 pad 2: GND -> /TX8/RF1
- C257 pad 1: /TX9/AGDC -> /TX8/RF2
- C257 pad 2: GND -> Net-(C257-Pad2)
- C258 pad 1: /TX9/HSEN1 -> GND
- C258 pad 2: GND -> +5VP
- C259 pad 1: /TX9/HSEN2 -> +5VP
- C260 pad 1: /TX9/RF2 -> Net-(C260-Pad1)
- C261 pad 1: GND -> +5VP
- C261 pad 2: /TX9/RF1 -> GND
- C262 pad 1: /TX9/RF2 -> /TX9/VDD_D
- C262 pad 2: Net-(C262-Pad2) -> GND
- C263 pad 1: GND -> +5VP
- C263 pad 2: +5VP -> GND
- C264 pad 1: +5VP -> /TX9/VDD_D
- C265 pad 1: Net-(C265-Pad1) -> /TX9/VDD_A
- C266 pad 1: +5VP -> /TX9/VDD_RF
- C267 pad 1: /TX10/VDD_D -> /TX9/VDD_A
- C268 pad 1: +5VP -> /TX9/VDD_RF
- C269 pad 1: /TX10/VDD_D -> /TX9/VDD_AM
- C270 pad 1: /TX10/VDD_A -> Net-(C270-Pad1)
- C271 pad 1: /TX10/VDD_RF -> /TX9/VDD_AM
- C272 pad 1: /TX10/VDD_A -> /CLK4
- C273 pad 1: /TX10/VDD_RF -> /TX9/VPD2
- C274 pad 1: /TX10/VDD_AM -> Net-(C274-Pad1)
- C277 pad 1: /CLK5 -> /TX9/VDET1
- C278 pad 1: Net-(C278-Pad1) -> /TX9/VDET2
- C280 pad 1: /TX10/VDET1 -> Net-(C280-Pad1)
- C281 pad 1: /TX10/VDET2 -> /TX9/AGDC
- C282 pad 1: Net-(C282-Pad1) -> /TX9/AGDC
- C284 pad 1: /TX10/AGDC -> /TX9/HSEN1
- C285 pad 1: /TX10/AGDC -> /TX9/HSEN2
- C286 pad 1: /TX10/HSEN1 -> /TX9/RF2
- C287 pad 1: /TX10/HSEN2 -> GND
- C287 pad 2: GND -> /TX9/RF1
- C288 pad 1: /TX10/RF2 -> /TX9/RF2
- C288 pad 2: GND -> Net-(C288-Pad2)
- C289 pad 2: /TX10/RF1 -> +5VP
- C290 pad 1: /TX10/RF2 -> +5VP
- C290 pad 2: Net-(C290-Pad2) -> GND
- C39 pad 1: GND -> /DTRD
- C39 pad 2: +5VP -> /RES
- C40 pad 1: +5VP -> /TX1/VPD2
- C41 pad 1: Net-(C41-Pad1) -> GND
- C41 pad 2: GND -> +5VP
- C43 pad 1: /TX2/VDD_D -> Net-(C43-Pad1)
- C46 pad 1: /TX2/VDD_A -> +5VP
- C47 pad 1: /TX2/VDD_RF -> /TX2/VDD_D
- C50 pad 1: /TX2/VDD_AM -> /TX2/VDD_A
- C51 pad 1: Net-(C51-Pad1) -> /TX2/VDD_RF
- C53 pad 1: /CLK2 -> Net-(C53-Pad1)
- C54 pad 1: Net-(C54-Pad1) -> /TX2/VDD_AM
- C55 pad 1: Net-(C55-Pad1) -> /CLK2
- C56 pad 1: /TX2/VDET1 -> /TX2/VPD2
- C57 pad 1: /TX2/VDET2 -> Net-(C57-Pad1)
- C60 pad 1: /TX2/AGDC -> /TX2/VDET1
- C61 pad 1: /TX2/AGDC -> /TX2/VDET2
- C62 pad 1: /TX2/HSEN1 -> Net-(C62-Pad1)
- C63 pad 1: /TX2/HSEN2 -> Net-(C63-Pad1)
- C64 pad 1: /TX2/RF2 -> /TX2/AGDC
- C65 pad 1: GND -> /TX2/AGDC
- C65 pad 2: /TX2/RF1 -> GND
- C67 pad 1: GND -> /TX2/HSEN1
- C67 pad 2: +5VP -> GND
- C68 pad 1: +5VP -> /TX2/HSEN2
- C69 pad 1: Net-(C69-Pad1) -> /TX2/RF2
- C70 pad 1: +5VP -> GND
- C70 pad 2: GND -> /TX2/RF1
- C71 pad 1: /TX3/VDD_D -> /TX2/RF2
- C71 pad 2: GND -> Net-(C71-Pad2)
- C72 pad 1: +5VP -> GND
- C72 pad 2: GND -> +5VP
- C73 pad 1: /TX3/VDD_D -> +5VP
- C74 pad 1: /TX3/VDD_A -> Net-(C74-Pad1)
- C75 pad 1: /TX3/VDD_RF -> +5VP
- C76 pad 1: /TX3/VDD_A -> /TX3/VDD_D
- C77 pad 1: /TX3/VDD_RF -> +5VP
- C78 pad 1: /TX3/VDD_AM -> /TX3/VDD_D
- C79 pad 1: Net-(C79-Pad1) -> /TX3/VDD_A
- C80 pad 1: /TX3/VDD_AM -> /TX3/VDD_RF
- C81 pad 1: /CLK3 -> /TX3/VDD_A
- C82 pad 1: Net-(C82-Pad1) -> /TX3/VDD_RF
- C83 pad 1: Net-(C83-Pad1) -> /TX3/VDD_AM
- C84 pad 1: /TX3/VDET1 -> Net-(C84-Pad1)
- C85 pad 1: /TX3/VDET2 -> /TX3/VDD_AM
- C86 pad 1: Net-(C86-Pad1) -> /CLK3
- C87 pad 1: Net-(C87-Pad1) -> /TX3/VPD2
- C88 pad 1: /TX3/AGDC -> Net-(C88-Pad1)
- C89 pad 1: /TX3/AGDC -> Net-(C89-Pad1)
- C9 pad 1: +5VP -> /DEV1/3V3
- C91 pad 1: /TX3/HSEN2 -> /TX3/VDET1
- C92 pad 1: /TX3/RF2 -> /TX3/VDET2
- C93 pad 1: GND -> Net-(C93-Pad1)
- C93 pad 2: /TX3/RF1 -> GND
- C94 pad 1: /TX3/RF2 -> Net-(C94-Pad1)
- C94 pad 2: Net-(C94-Pad2) -> GND
- C95 pad 1: GND -> /TX3/AGDC
- C95 pad 2: +5VP -> GND
- C96 pad 1: +5VP -> /TX3/AGDC
- C98 pad 1: +5VP -> /TX3/HSEN1
- C99 pad 1: /TX4/VDD_D -> /TX3/HSEN2
- D14 pad 1: /TX2/HSEN2 -> /TX2/HSEN1
- D14 pad 3: Net-(C59-Pad1) -> Net-(C62-Pad1)
- D15 pad 1: Net-(D15-Pad1) -> /TX2/HSEN2
- D15 pad 2: /TX2/RF1 -> Net-(D15-Pad2)
- D17 pad 2: /TX2/GRN -> /TX2/RF1
- D18 pad 1: /TX2/BLU -> Net-(D18-Pad1)
- D18 pad 2: Net-(D18-Pad2) -> /TX2/RED
- D19 pad 1: /TX3/HSEN1 -> Net-(D19-Pad1)
- D19 pad 2: Net-(D19-Pad2) -> /TX2/GRN
- D20 pad 1: /TX3/HSEN2 -> /TX2/BLU
- D21 pad 1: Net-(D21-Pad1) -> /TX3/HSEN1
- D21 pad 2: /TX3/RF1 -> Net-(D21-Pad2)
- D22 pad 1: Net-(D22-Pad1) -> /TX3/HSEN2
- D22 pad 2: /TX3/RED -> Net-(D22-Pad2)
- D24 pad 1: /TX3/BLU -> Net-(D24-Pad1)
- D24 pad 2: Net-(D24-Pad2) -> /TX3/RF1
- D25 pad 1: /TX4/HSEN1 -> Net-(D25-Pad1)
- D25 pad 2: Net-(D25-Pad2) -> /TX3/RED
- D26 pad 1: /TX4/HSEN2 -> Net-(D26-Pad1)
- D26 pad 2: Net-(D26-Pad2) -> /TX3/GRN
- D27 pad 1: Net-(D27-Pad1) -> /TX3/BLU
- D27 pad 2: /TX4/RF1 -> Net-(D27-Pad2)
- D28 pad 1: Net-(D28-Pad1) -> /TX4/HSEN1
- D28 pad 2: /TX4/RED -> Net-(D28-Pad2)
- D29 pad 1: Net-(D29-Pad1) -> /TX4/HSEN2
- D29 pad 2: /TX4/GRN -> Net-(D29-Pad2)
- D31 pad 1: /TX5/HSEN1 -> Net-(D31-Pad1)
- D31 pad 2: Net-(D31-Pad2) -> /TX4/RF1
- D32 pad 1: /TX5/HSEN2 -> Net-(D32-Pad1)
- D32 pad 2: Net-(D32-Pad2) -> /TX4/RED
- D33 pad 2: /TX5/RF1 -> /TX4/GRN
- D34 pad 1: Net-(D34-Pad1) -> /TX4/BLU
- D34 pad 2: /TX5/RED -> Net-(D34-Pad2)
- D35 pad 1: Net-(D35-Pad1) -> /TX5/HSEN1
- D35 pad 2: /TX5/GRN -> Net-(D35-Pad2)
- D36 pad 1: /TX5/BLU -> /TX5/HSEN2
- D38 pad 1: /TX6/HSEN2 -> Net-(D38-Pad1)
- D38 pad 2: Net-(D38-Pad2) -> /TX5/RF1
- D39 pad 2: /TX6/RF1 -> /TX5/RED
- D40 pad 2: /TX6/RED -> /TX5/GRN
- D41 pad 1: Net-(D41-Pad1) -> /TX5/BLU
- D41 pad 2: /TX6/GRN -> Net-(D41-Pad2)
- D42 pad 1: /TX6/BLU -> /TX6/HSEN1
- D43 pad 1: /TX7/HSEN1 -> /TX6/HSEN2
- D43 pad 3: Net-(C198-Pad1) -> Net-(C187-Pad1)
- D45 pad 2: /TX7/RF1 -> /TX6/RF1
- D46 pad 2: /TX7/RED -> /TX6/RED
- D47 pad 2: /TX7/GRN -> /TX6/GRN
- D48 pad 1: /TX7/BLU -> /TX6/BLU
- D49 pad 1: /TX8/HSEN1 -> /TX7/HSEN1
- D49 pad 3: Net-(C226-Pad1) -> Net-(C217-Pad1)
- D50 pad 1: /TX8/HSEN2 -> /TX7/HSEN2
- D50 pad 3: Net-(C227-Pad1) -> Net-(C218-Pad1)
- D52 pad 2: /TX8/RED -> /TX7/RF1
- D53 pad 2: /TX8/GRN -> /TX7/RED
- D54 pad 1: /TX8/BLU -> Net-(D54-Pad1)
- D54 pad 2: Net-(D54-Pad2) -> /TX7/GRN
- D55 pad 1: /TX9/HSEN1 -> /TX7/BLU
- D56 pad 1: /TX9/HSEN2 -> /TX8/HSEN1
- D56 pad 3: Net-(C255-Pad1) -> Net-(C248-Pad1)
- D57 pad 1: Net-(D57-Pad1) -> /TX8/HSEN2
- D57 pad 2: /TX9/RF1 -> Net-(D57-Pad2)
- D59 pad 2: /TX9/GRN -> /TX8/RF1
- D60 pad 1: /TX9/BLU -> Net-(D60-Pad1)
- D60 pad 2: Net-(D60-Pad2) -> /TX8/RED
- D61 pad 1: /TX10/HSEN1 -> Net-(D61-Pad1)
- D61 pad 2: Net-(D61-Pad2) -> /TX8/GRN
- D62 pad 1: /TX10/HSEN2 -> /TX8/BLU
- D63 pad 1: Net-(D63-Pad1) -> /TX9/HSEN1
- D63 pad 2: /TX10/RF1 -> Net-(D63-Pad2)
- D64 pad 1: Net-(D64-Pad1) -> /TX9/HSEN2
- D64 pad 2: /TX10/RED -> Net-(D64-Pad2)
- D66 pad 1: /TX10/BLU -> Net-(D66-Pad1)
- D66 pad 2: Net-(D66-Pad2) -> /TX9/RF1
- J10 pad 1: /TX2/HSEN2 -> /TX2/MISO
- J10 pad 2: GND -> +5VP
- J11 pad 1: Net-(J11-Pad1) -> +5VP
- J11 pad 2: Net-(J11-Pad2) -> /TX2/LSEN2
- J12 pad 1: /TX3/MISO -> Net-(J12-Pad1)
- J12 pad 2: +5VP -> Net-(J12-Pad2)
- J13 pad 1: /TX3/HSEN2 -> /TX3/MISO
- J13 pad 2: GND -> +5VP
- J14 pad 1: Net-(J14-Pad1) -> +5VP
- J14 pad 2: Net-(J14-Pad2) -> /TX3/LSEN2
- J15 pad 1: /TX4/MISO -> Net-(J15-Pad1)
- J15 pad 2: +5VP -> Net-(J15-Pad2)
- J16 pad 1: /TX4/HSEN2 -> /TX4/MISO
- J16 pad 2: GND -> +5VP
- J17 pad 1: Net-(J17-Pad1) -> +5VP
- J17 pad 2: Net-(J17-Pad2) -> /TX4/LSEN2
- J18 pad 1: /TX5/MISO -> Net-(J18-Pad1)
- J18 pad 2: +5VP -> Net-(J18-Pad2)
- J19 pad 1: /TX5/HSEN2 -> /TX5/MISO
- J19 pad 2: GND -> +5VP
- J20 pad 1: Net-(J20-Pad1) -> +5VP
- J20 pad 2: Net-(J20-Pad2) -> /TX5/LSEN2
- J21 pad 1: /TX6/MISO -> Net-(J21-Pad1)
- J21 pad 2: +5VP -> Net-(J21-Pad2)
- J22 pad 1: /TX6/HSEN2 -> /TX6/MISO
- J22 pad 2: GND -> +5VP
- J23 pad 1: Net-(J23-Pad1) -> +5VP
- J23 pad 2: Net-(J23-Pad2) -> /TX6/LSEN2
- J24 pad 1: /TX7/MISO -> Net-(J24-Pad1)
- J24 pad 2: +5VP -> Net-(J24-Pad2)
- J25 pad 1: /TX7/HSEN2 -> /TX7/MISO
- J25 pad 2: GND -> +5VP
- J26 pad 1: Net-(J26-Pad1) -> +5VP
- J26 pad 2: Net-(J26-Pad2) -> /TX7/LSEN2
- J27 pad 1: /TX8/MISO -> Net-(J27-Pad1)
- J27 pad 2: +5VP -> Net-(J27-Pad2)
- J28 pad 1: /TX8/HSEN2 -> /TX8/MISO
- J28 pad 2: GND -> +5VP
- J29 pad 1: Net-(J29-Pad1) -> +5VP
- J29 pad 2: Net-(J29-Pad2) -> /TX8/LSEN2
- J30 pad 1: /TX9/MISO -> Net-(J30-Pad1)
- J30 pad 2: +5VP -> Net-(J30-Pad2)
- J31 pad 1: /TX9/HSEN2 -> /TX9/MISO
- J31 pad 2: GND -> +5VP
- J32 pad 1: Net-(J32-Pad1) -> +5VP
- J32 pad 2: Net-(J32-Pad2) -> /TX9/LSEN2
- J33 pad 1: /TX10/MISO -> Net-(J33-Pad1)
- J33 pad 2: +5VP -> Net-(J33-Pad2)
- J34 pad 1: /TX10/HSEN2 -> /TX10/MISO
- J34 pad 2: GND -> +5VP
- J35 pad 1: Net-(J35-Pad1) -> +5VP
- J35 pad 2: Net-(J35-Pad2) -> /TX10/LSEN2
- J7 pad 1: /TX1/HSEN2 -> +5VP
- J7 pad 2: GND -> /TX1/LSEN2
- J9 pad 1: /TX2/MISO -> GND
- J9 pad 2: +5VP -> +5V
- J9 pad 3: /TX2/SCK -> /ENCA
- J9 pad 4: /TX2/MOSI -> /ENCB
- MT1 pad 1: (no net) -> Net-(MT1-Pad1)
- MT2 pad 1: (no net) -> Net-(MT2-Pad1)
- MT3 pad 1: (no net) -> Net-(MT3-Pad1)
- MT4 pad 1: (no net) -> Net-(MT4-Pad1)
- Q4 pad 3: /TX -> /TXT
- Q5 pad 3: /RX -> /RXT
- R100 pad 1: /TX8/VDET1 -> /TX7/RES
- R100 pad 2: Net-(C226-Pad1) -> +5VP
- R101 pad 1: /TX8/VDET2 -> /TX7/VDET1
- R101 pad 2: Net-(C227-Pad1) -> Net-(C217-Pad1)
- R102 pad 1: /TX8/VDET1 -> /TX7/VDET2
- R102 pad 2: GND -> Net-(C218-Pad1)
- R103 pad 1: /TX8/VDET2 -> /TX7/VDET1
- R105 pad 2: GND -> /TX7/RF2
- R107 pad 1: Net-(D54-Pad2) -> Net-(D54-Pad1)
- R108 pad 1: /SDAP -> Net-(D55-Pad2)
- R108 pad 2: +5VP -> GND
- R109 pad 1: /SCLP -> /SDAP
- R110 pad 1: /TX9/RES -> /SCLP
- R111 pad 1: /TX9/VDET1 -> /TX8/LSEN2
- R111 pad 2: Net-(C254-Pad1) -> /TX8/VPD2
- R113 pad 1: /TX9/VDET1 -> /TX8/RES
- R113 pad 2: GND -> +5VP
- R114 pad 1: /TX9/VDET2 -> /TX8/VDET1
- R114 pad 2: GND -> Net-(C248-Pad1)
- R115 pad 1: Net-(D57-Pad1) -> /TX8/VDET2
- R115 pad 2: /TX9/RF2 -> Net-(C249-Pad1)
- R116 pad 1: Net-(D58-Pad1) -> /TX8/VDET1
- R118 pad 1: Net-(D60-Pad2) -> Net-(D59-Pad1)
- R118 pad 2: GND -> /TX8/RF2
- R119 pad 1: /SDAP -> Net-(D60-Pad1)
- R119 pad 2: +5VP -> GND
- R120 pad 1: /SCLP -> Net-(D61-Pad1)
- R120 pad 2: +5VP -> GND
- R121 pad 1: /TX10/RES -> Net-(D62-Pad2)
- R121 pad 2: +5VP -> GND
- R122 pad 1: /TX10/VDET1 -> /SDAP
- R122 pad 2: Net-(C282-Pad1) -> +5VP
- R123 pad 1: /TX10/VDET2 -> /SCLP
- R123 pad 2: Net-(C283-Pad1) -> +5VP
- R124 pad 1: /TX10/VDET1 -> /TX9/LSEN2
- R124 pad 2: GND -> /TX9/VPD2
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Routing:
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Other:
- board size 270 x 125 mm -> 270 x 121 mm
- board text added: "3V3 MOSI GND"
- board text added: "5V/2A"
- board text added: "Encoder (5V)"
- board text added: "GND 3V3 SDA2 SCL2"
- board text added: "GND 5V ENCA ENCB"
- board text added: "GND 5V MISO MOSI SCK SDCS"
- board text added: "GND MOSI 5V"
- board text added: "I2C Ports (3.3V)"
- board text added: "MISO SCK CSS"
- board text added: "NFCPower10 - YSO - Rev 2"
- board text added: "OLED Display I2C Port (5V)"
- board text added: "SD Card SPI Port (5V)"
- board text added: "SPI Port (3.3V)"
- board text removed: "5V/3A"
- board text removed: "CS SCK MOSI MISO +5V GND"
- board text removed: "GND MOSI +5V"
- board text removed: "HSEN1"
- board text removed: "HSEN2"
- board text removed: "NFCPower10 - YSO"
- board text removed: "OLED Display I2C Port"
- board text removed: "RED"
- board text removed: "RF ON"
- board text removed: "RX"
- board text removed: "RXP"
- board text removed: "SCK"
- board text removed: "SD Card SPI Port"
- board text removed: "SDA SCL +5V GND"
- board text removed: "TX"
- board text removed: "TX1"
- board text removed: "TX10"
- board text removed: "TX2"
- board text removed: "TX3"
- board text removed: "TX4"
- board text removed: "TX5"
- board text removed: "TX6"
- board text removed: "TX7"
- board text removed: "TX8"
- board text removed: "TX9"
- board text removed: "TXP"
